File: Light_Sensor_schematic/Light_Sensor_schematic.sch (KiCad schematic (older format))
At the start: 21 parts, among them IC1 TSL237S-LF, J1 Conn_01x03, J3 Conn_01x04_Male, U1 STM32L432KCUx, U2 STDC14, U3 TG-3541CE

Commit message: Lab 8
Connections:
- net VDD: no longer C1.1
- net sensor_pwr: now also C1.1
Changed lines of the file:
@@
 tsl237_freq
-$Comp
-L power:VDD #PWR0118
-U 1 1 62401D92
-P 3950 5150
-F 0 "#PWR0118" H 3950 5000 50  0001 C CNN
-F 1 "VDD" H 3965 5323 50  0000 C CNN
-F 2 "" H 3950 5150 50  0001 C CNN
-F 3 "" H 3950 5150 50  0001 C CNN
-	1    3950 5150
-	1    0    0    -1
-$EndComp
 $Comp
 L pspice:CAP C1
@@
 Wire Wire Line
 	1950 2200 1950 2400
+Text Label 3950 5150 0    50   ~ 0
+sensor_pwr
 $EndSCHEMATC
